Commit message: updated to make ros2_control work for duco robot

File: src/duco_gcr5_910_moveit_config/config/gcr5_910.ros2_control.xacro (robot description, xacro)
@@ -1,10 +1,20 @@
 <?xml version="1.0"?>
 <robot xmlns:xacro="http://www.ros.org/wiki/xacro">
-    <xacro:macro name="gcr5_910_ros2_control" params="name initial_positions_file">
-        <xacro:property name="initial_positions" value="${load_yaml(initial_positions_file)['initial_positions']}"/>
+    <xacro:macro name="gcr5_910_ros2_control" params="name initial_positions_file robot_ip:=192.168.1.10 robot_port:=7003 use_fake_hardware:=false">
+        <xacro:property name="initial_positions" value="${xacro.load_yaml(initial_positions_file)['initial_positions']}"/>
         <ros2_control name="${name}" type="system">
             <hardware>
-                <!-- By default, set up controllers for simulation. This won't work on real hardware -->
-                <plugin>mock_components/GenericSystem</plugin>
+                <xacro:if value="${use_fake_hardware}">
+                    <!-- Simulation mode with mock components -->
+                    <plugin>mock_components/GenericSystem</plugin>
+                    <param name="mock_sensor_commands">false</param>
+                    <param name="state_following_offset">0.0</param>
+                </xacro:if>
+                <xacro:unless value="${use_fake_hardware}">
+                    <!-- Real DUCO hardware interface -->
+                    <plugin>duco_hardware/DucoHardwareInterface</plugin>
+                    <param name="robot_ip">${robot_ip}</param>
+                    <param name="robot_port">${robot_port}</param>
+                </xacro:unless>
             </hardware>
             <joint name="arm_1_joint_1">

File: src/duco_gcr5_910_moveit_config/config/gcr5_910.urdf.xacro (robot description, xacro)
@@ -2,8 +2,11 @@
 <robot xmlns:xacro="http://www.ros.org/wiki/xacro" name="gcr5_910">
     <xacro:arg name="initial_positions_file" default="initial_positions.yaml" />
+    <xacro:arg name="robot_ip" default="192.168.1.10" />
+    <xacro:arg name="robot_port" default="7003" />
+    <xacro:arg name="use_fake_hardware" default="false" />
     <!-- Import gcr5_910 urdf file -->
     <xacro:include filename="$(find duco_support)/urdf/duco_gcr5_910.urdf" />
     <!-- Import control_xacro -->
     <xacro:include filename="gcr5_910.ros2_control.xacro" />
-    <xacro:gcr5_910_ros2_control name="FakeSystem" initial_positions_file="$(arg initial_positions_file)"/>
+    <xacro:gcr5_910_ros2_control name="FakeSystem" initial_positions_file="$(arg initial_positions_file)" robot_ip="$(arg robot_ip)" robot_port="$(arg robot_port)" use_fake_hardware="$(arg use_fake_hardware)"/>
 </robot>
